File: C64Saver2-addon/C64Saver2-addon.sch (KiCad schematic (older format))
At the start: 14 parts, among them J1 Conn_01x12_Female, J2 Conn_01x07_Female, J3 Conn_01x04_Male, SW1 SW_Push, SW2 SW_Push, U1 ProMicro, U3 INA219, U4 VO615A-5, U5 4N25, U6 ADuM1200BR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

Commit message: Tidy up project libraries. Relative paths
Parts:
- removed U1: ProMicro, promicro:ProMicro, symbol ProMicro
- added U3: ProMicro, promicro:ProMicro, symbol ProMicro
- U1: renamed from U3; footprint ina216:ina216board -> ina219:ina219
- renumbered SW2 to SW1, SW1 to SW2, U6 to U2, U7 to U6
Changed lines of the file:
@@
 LIBS:contrib
 LIBS:valves
+LIBS:ina219
 LIBS:promicro
-LIBS:ina219
 LIBS:C64Saver2-addon-cache
 EELAYER 25 0
@@
 $EndDescr
 $Comp
-L ProMicro U1
-U 1 1 5B217998
-P 7550 3900
-F 0 "U1" H 7550 4850 60  0000 C CNN
-F 1 "ProMicro" H 7550 3350 60  0000 C CNN
-F 2 "promicro:ProMicro" H 7650 2850 60  0001 C CNN
-F 3 "" H 7650 2850 60  0000 C CNN
-	1    7550 3900
-	1    0    0    -1
-$EndComp
-$Comp
-L INA219 U3
+L INA219 U1
 U 1 1 5B218B38
 P 2100 4200
-F 0 "U3" H 2100 5150 60  0000 C CNN
+F 0 "U1" H 2100 5150 60  0000 C CNN
 F 1 "INA219" H 1750 4250 60  0000 C CNN
-F 2 "ina216:ina216board" H 2200 3150 60  0001 C CNN
+F 2 "ina219:ina219" H 2200 3150 60  0001 C CNN
 F 3 "" H 2200 3150 60  0000 C CNN
 	1    2100 4200
@@
 $EndComp
 $Comp
-L 4N25 U7
+L 4N25 U6
 U 1 1 5B21CB3E
 P 9300 4350
-F 0 "U7" H 9100 4550 50  0000 L CNN
+F 0 "U6" H 9100 4550 50  0000 L CNN
 F 1 "4N25" H 9300 4550 50  0000 L CNN
 F 2 "TO_SOT_Packages_SMD:SOT-23-6" H 9100 4150 50  0001 L CIN
@@
 VIN-
 $Comp
-L ADuM1200BR U6
+L ADuM1200BR U2
 U 1 1 5B21CDC6
 P 4850 3750
-F 0 "U6" H 4500 4150 50  0000 L CNN
+F 0 "U2" H 4500 4150 50  0000 L CNN
 F 1 "ADuM1200BR" H 4800 4150 50  0000 L CNN
 F 2 "Housings_SOIC:SOIC-8_3.9x4.9mm_Pitch1.27mm" H 4850 3750 50  0001 C CIN
@@
 $EndComp
 $Comp
-L SW_Push SW1
+L SW_Push SW2
 U 1 1 5B22D489
 P 6350 4100
-F 0 "SW1" H 6400 4200 50  0000 L CNN
+F 0 "SW2" H 6400 4200 50  0000 L CNN
 F 1 "SW_Push" H 6350 4040 50  0000 C CNN
 F 2 "Buttons_Switches_THT:SW_PUSH_6mm_h13mm" H 6350 4300 50  0001 C CNN
@@
 $EndComp
 $Comp
-L SW_Push SW2
+L SW_Push SW1
 U 1 1 5B22D5E5
 P 6350 3850
-F 0 "SW2" H 6400 3950 50  0000 L CNN
+F 0 "SW1" H 6400 3950 50  0000 L CNN
 F 1 "SW_Push" H 6350 3790 50  0000 C CNN
 F 2 "Buttons_Switches_THT:SW_PUSH_6mm_h13mm" H 6350 4050 50  0001 C CNN
@@
 	1    0    0    -1
 $EndComp
+$Comp
+L ProMicro U3
+U 1 1 5B263A73
+P 7550 3900
+F 0 "U3" H 7550 4850 60  0000 C CNN
+F 1 "ProMicro" H 7550 3350 60  0000 C CNN
+F 2 "promicro:ProMicro" H 7650 2850 60  0001 C CNN
+F 3 "" H 7650 2850 60  0000 C CNN
+	1    7550 3900
+	1    0    0    -1
+$EndComp
