File: C64Saver2-addon/C64Saver2-addon.sch (KiCad schematic (older format))
At the start: 25 parts, among them J1 Conn_01x12_Female, J2 Conn_01x07_Female, J3 OLED_128x32_Conn_01x04_Male, SW1 SW_Push, SW2 SW_Push, U1 INA219xIDR-SOIC, U2 ISO1541D, U3 ProMicro, U4 4N25, U5 4N25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

Commit message: saver 2.0beta - addon 1.0beta
Other:
- note added: "1.0beta"
Changed lines of the file:
@@
 Wire Wire Line
 	6100 2850 6100 2800
+Text Notes 10650 7650 0    60   ~ 0
+1.0beta
 $EndSCHEMATC

Commit message: eddited schematic of addon board
Parts:
- removed R7: 560, Resistors_SMD:R_0603_HandSoldering, symbol R_Small
- added U?: AP1117-50, TO_SOT_Packages_SMD:SOT-223-3Lead_TabPin2, symbol AP1117-50
Connections:
- wire segments 111 -> 115
Other:
- note added: "1.0"
- note removed: "1.0beta"
- moved on the sheet: C1, C3, C4, C5, D1, J3, R1, R3, R5, R6, R8, SW1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
