File: C64Saver2-addon/_saved_C64Saver2-addon.sch (KiCad schematic (older format))
At the start: 29 parts, among them J1 Conn_01x12_Female, J2 Conn_01x07_Female, J3 OLED_128x32_Conn_01x04_Male, SW1 SW_Push, SW2 SW_Push, U1 INA219xIDR-SOIC, U2 ISO1541D, U3 ProMicro, U4 PC817, U6 ACS712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

Commit message: SOP4 model
Parts:
- removed U4, U8: PC817, sop:SOP4-WIDE, symbol PC817
- added U4, U5: TLP291, sop:SOP4, symbol TLP291
Connections:
- net #OVERVOLTAGE: now also U5.4
- net GND: now also U4.3, U5.3
- net HOLD: now also U4.4
- net OVERVOLTAGE: now also U5.2
- net PGATE: now also U4.2
- net VIN-: now also U4.1
- net at R3.1: now also U5.1
Changed lines of the file:
@@
 	1    0    0    -1
 $EndComp
+Wire Wire Line
+	4500 5050 4550 5050
 $Comp
-L PC817 U8
-U 1 1 5B3C18C9
+L TLP291 U4
+U 1 1 5B3D5BA2
 P 4850 5150
-F 0 "U8" H 4650 5350 50  0000 L CNN
-F 1 "PC817" H 4850 5350 50  0000 L CNN
-F 2 "sop:SOP4-WIDE" H 4650 4950 50  0001 L CIN
+F 0 "U4" H 4650 5350 50  0000 L CNN
+F 1 "TLP291" H 4850 5350 50  0000 L CNN
+F 2 "sop:SOP4" H 4650 4950 50  0001 L CIN
 F 3 "" H 4850 5150 50  0001 L CNN
 	1    4850 5150
@@
 $EndComp
 $Comp
-L PC817 U4
-U 1 1 5B3C21F6
+L TLP291 U5
+U 1 1 5B3D5E18
 P 4850 5900
-F 0 "U4" H 4650 6100 50  0000 L CNN
-F 1 "PC817" H 4850 6100 50  0000 L CNN
-F 2 "sop:SOP4-WIDE" H 4650 5700 50  0001 L CIN
+F 0 "U5" H 4650 6100 50  0000 L CNN
+F 1 "TLP291" H 4850 6100 50  0000 L CNN
+F 2 "sop:SOP4" H 4650 5700 50  0001 L CIN
 F 3 "" H 4850 5900 50  0001 L CNN
 	1    4850 5900
 	1    0    0    -1
 $EndComp
-Wire Wire Line
-	4500 5050 4550 5050
 $EndSCHEMATC
