File: C64Saver2/C64Saver2.kicad_pcb (KiCad board)
At the start: 2 copper layers, 45.7 x 35.6 mm, 21 parts, among them J1 Conn_01x04, J2 Conn_01x12, J3 Conn_01x12, J6 Conn_01x04, Q1 2N7002, Q2 Q_PMOS_GDS

Commit message: Name, revision, author on silk.s
Other:
- board text added: "C64 Saver 2 Rev 2.0 BWACK 2018"
Changed lines of the file:
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@@
     (area 102.794999 91.364999 148.665001 127.075001)
     (thickness 1.6)
-    (drawings 23)
+    (drawings 24)
     (tracks 136)
     (zones 0)
@@
     )
   )
+  (gr_text "C64 Saver 2\nRev 2.0 BWACK 2018" (at 125.349 120.269) (layer F.SilkS)
+    (effects (font (size 1.2 1.5) (thickness 0.3)))
+  )
   (dimension 45.72 (width 0.3) (layer Dwgs.User)
     (gr_text "45,720 mm" (at 125.73 137.24) (layer Dwgs.User)
@@
     (effects (font (size 1.25 1.25) (thickness 0.3)) (justify mirror))
   )
-  (gr_text OUT (at 139.446 120.65) (layer F.SilkS)
+  (gr_text OUT (at 138.6332 118.7958) (layer F.SilkS)
     (effects (font (size 1.5 1.5) (thickness 0.3)))
   )
-  (gr_text IN (at 110.744 120.65) (layer F.SilkS)
+  (gr_text IN (at 111.76 118.6688) (layer F.SilkS)
     (effects (font (size 1.5 1.5) (thickness 0.3)))
   )
