File: C64Saver2/C64Saver2.kicad_pcb (KiCad board)
At the start: 2 copper layers, 45.7 x 35.6 mm, 21 parts, among them J1 Conn_01x04, J2 Conn_01x12, J3 Conn_01x12, J6 Conn_01x04, Q1 2N7002, Q2 Q_PMOS_GDS

Commit message: saver 2.0beta - addon 1.0beta
Other:
- board text added: "C64 Saver Rev 2.0beta BWACK 2018"
- board text removed: "C64 Saver 2 Rev 2.0 BWACK 2018"
Changed lines of the file:
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@@
     (links 50)
     (no_connects 0)
-    (area 100.855 89.13238 160.25 138.590001)
+    (area 102.794999 91.364999 148.665001 127.075001)
     (thickness 1.6)
     (drawings 25)
@@
     (arrow2b (pts (xy 156.591 91.44) (xy 157.177421 92.566504)))
   )
-  (gr_text "C64 Saver 2\nRev 2.0 BWACK 2018" (at 125.349 120.269) (layer F.SilkS)
+  (gr_text "C64 Saver\nRev 2.0beta BWACK 2018" (at 125.349 120.269) (layer F.SilkS)
     (effects (font (size 1.2 1.5) (thickness 0.3)))
   )

Commit message: added gnd, 5x 9vac pins, moved c1 closer to input circuit
Parts:
- J3: value Conn_01x12 -> Conn_01x07; footprint Pin_Headers:Pin_Header_Straight_1x12_Pitch2.54mm -> Pin_Headers:Pin_Header_Straight_1x07_Pitch2.54mm
- moved C1 4.32 mm to (118.1, 99.6), turned to 180 degrees
Connections:
- net 9VAC2 renamed /9VAC2
- C1 pad 1: /VCC1+ -> /VCC1-
- J1 pad 3: 9VAC1 -> /9VAC1
- J2 pad 1: /VCC1+ -> GND
- J3 pad 1: GND -> /9VAC1
- J3 pad 2: GND -> /9VAC1
- J3 pad 3: GND -> /9VAC1'
- J3 pad 4: 9VAC1 -> /9VAC1'
- J6 pad 2: 9VAC1 -> /9VAC1'
Routing:
- net 9VAC1: track 64.0 -> 0.00 mm
- net /9VAC1': track 0.00 -> 40.4 mm, vias 0 -> 2
- net GND: track 124.0 -> 91.2 mm
- net /9VAC1: track 0.00 -> 17.3 mm
- net /VCC1+: track 27.9 -> 23.5 mm
- net /VCC1-: track 23.6 -> 21.8 mm
- net OVERVOLTAGE: track 32.1 -> 33.6 mm
Other:
- board text added: "C64 Saver Rev 2.0 BWACK 2018"
- board text removed: "C64 Saver Rev 2.0beta BWACK 2018"

Commit message: fit to hammond1591, larger board.
Parts:
- added REF**: hammond1591XXLGY_pcb, hammond1591:hammond1591XXLGY_pcb, F.Cu at (59.3, 86.1)
Changed lines of the file:
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@@
 (kicad_pcb (version 4) (host pcbnew 4.0.7)
   (general
-    (links 49)
+    (links 0)
     (no_connects 0)
-    (area 102.794999 91.364999 148.665001 127.075001)
+    (area 44.8652 35.111999 164.441 138.590001)
     (thickness 1.6)
     (drawings 25)
     (tracks 117)
     (zones 0)
-    (modules 21)
+    (modules 22)
     (nets 12)
   )
@@
   )
   (setup
-    (last_trace_width 0.5)
+    (last_trace_width 0.25)
     (user_trace_width 0.5)
     (user_trace_width 1)
@@
     )
   )
+  (module hammond1591:hammond1591XXLGY_pcb (layer F.Cu)
+    (at 59.2582 86.0552)
+    (fp_text reference REF** (at 10.16 1.27) (layer Eco1.User)
+      (effects (font (size 1 1) (thickness 0.15)))
+    )
+    (fp_text value hammond1591XXLGY_pcb (at 17.78 2.54) (layer Eco1.User)
+      (effects (font (size 1 1) (thickness 0.15)))
+    )
+    (fp_circle (center 14.9 -10.25) (end 16.65 -10.25) (layer Eco1.User) (width 0.15))
+    (fp_line (start 7.62 -7.62) (end 7.62 0) (layer Eco1.User) (width 0.15))
+    (fp_line (start 0 -7.62) (end 7.62 -7.62) (layer Eco1.User) (width 0.15))
+    (fp_line (start 72.39 -7.62) (end 72.39 0) (layer Eco1.User) (width 0.15))
+    (fp_line (start 80.01 -7.62) (end 72.39 -7.62) (layer Eco1.User) (width 0.15))
+    (fp_line (start 72.39 -43.18) (end 80.01 -43.18) (layer Eco1.User) (width 0.15))
+    (fp_line (start 72.39 -50.8) (end 72.39 -43.18) (layer Eco1.User) (width 0.15))
+    (fp_line (start 7.62 -43.18) (end 7.62 -50.8) (layer Eco1.User) (width 0.15))
+    (fp_line (start 0 -43.18) (end 7.62 -43.18) (layer Eco1.User) (width 0.15))
+    (fp_line (start 0 -7.75) (end 0 -43.25) (layer Eco1.User) (width 0.15))
+    (fp_line (start 7.75 0) (end 72.25 0) (layer Eco1.User) (width 0.15))
+    (fp_line (start 7.75 -51) (end 72.25 -51) (layer Eco1.User) (width 0.15))
+    (fp_line (start 80 -7.75) (end 80 -43.25) (layer Eco1.User) (width 0.15))
+    (fp_circle (center 65.1 -10.25) (end 66.85 -10.25) (layer Eco1.User) (width 0.15))
+    (fp_circle (center 14.9 -40.75) (end 16.65 -40.75) (layer Eco1.User) (width 0.15))
+    (fp_circle (center 65.1 -40.75) (end 66.85 -40.75) (layer Eco1.User) (width 0.15))
+  )
   (gr_text "C64 Saver\nRev 2.0 BWACK 2018" (at 125.349 120.269) (layer F.SilkS)
