File: addon board 1.0/C64Saver2-addon.kicad_pcb (KiCad board)
At the start: 2 copper layers, 43.9 x 29 mm, 39 parts, among them CON1 AVR-ISP-6, J1 Conn_01x08_Female, J2 Conn_01x08_Female, J3 OLED_128x32_Conn_01x04_Male, J4 Conn_01x04_Female, SW1 SW_Push, U1 INA219xIDR-SOIC, U2 ISO1541D, U3 ATTINY85-20SU, U4 TLP291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

Commit message: Release 2.1 and addon 1.0
Parts:
- C1: footprint Capacitors_SMD:C_1210_HandSoldering -> Capacitors_Tantalum_SMD:CP_Tantalum_Case-X_EIA-7343-43_Reflow
- R2: footprint Resistors_SMD:R_2010_HandSoldering -> Resistors_SMD:R_2512_HandSoldering
- moved D1 1.53 mm to (149.5, 107.4), turned to 0 degrees
- moved C5 1.02 mm to (151.2, 100.6)
- moved R1 1.02 mm to (151.3, 97.8)
- moved J3 0.89 mm to (142.2, 99.4)
- moved R12 0.76 mm to (146.5, 100.6)
- moved R8 0.76 mm to (146.5, 97.8)
- moved C1 0.61 mm to (145.5, 103.8)
- moved CON1 0.38 mm to (142.5, 85.0)
- moved R2 0.34 mm to (171.1, 89.5), turned to 0 degrees
- moved U7 0.26 mm to (154.1, 107.0)
- moved C10 0.25 mm to (154.0, 103.4)
Connections:
- J1 pad 1: /VIN+ -> VIN-
- J1 pad 2: /VIN+ -> VIN-
- J1 pad 3: /VIN+ -> VIN-
- J1 pad 4: /VIN+ -> VIN-
- J1 pad 5: VIN- -> /VIN+
- J1 pad 6: VIN- -> /VIN+
- J1 pad 7: VIN- -> /VIN+
- J1 pad 8: VIN- -> /VIN+
- J2 pad 1: /9VAC1+ -> /9VAC1-
- J2 pad 2: /9VAC1+ -> /9VAC1-
- J2 pad 3: /9VAC1+ -> /9VAC1-
- J2 pad 4: /9VAC1+ -> /9VAC1-
- J2 pad 5: /9VAC1- -> /9VAC1+
- J2 pad 6: /9VAC1- -> /9VAC1+
- J2 pad 7: /9VAC1- -> /9VAC1+
- J2 pad 8: /9VAC1- -> /9VAC1+
Routing:
- net /9VAC1+: track 41.6 -> 67.2 mm
- net VIN-: track 76.2 -> 67.4 mm
- net /9VAC1-: track 38.4 -> 32.8 mm
- net +5V: track 102.7 -> 97.4 mm
- net Net-(C1-Pad2): track 8.98 -> 11.4 mm
- net /VIN+: track 20.1 -> 18.2 mm
- net /SCL1: track 66.5 -> 65.2 mm
- net /HOLD_: track 11.9 -> 10.9 mm
- net /SDA1: track 61.7 -> 61.1 mm
- net /HOLD: track 3.60 -> 3.05 mm
Other:
- board text added: "1.0"
- board text added: "2017-07-23"
- board text added: "C64 Saver addon board"
