File: addon board 1.0/C64Saver2-addon.sch (KiCad schematic (older format))
At the start: 38 parts, among them CON1 AVR-ISP-6, J1 Conn_01x08_Female, J2 Conn_01x08_Female, J3 OLED_128x32_Conn_01x04_Male, J4 Conn_01x04_Female, SW1 SW_Push, U1 INA219xIDR-SOIC, U2 ISO1541D, U3 ATTINY85-20SU, U4 TLP291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

Commit message: Release 2.1 and addon 1.0
Parts:
- C1: footprint Capacitors_SMD:C_1210_HandSoldering -> Capacitors_Tantalum_SMD:CP_Tantalum_Case-X_EIA-7343-43_Reflow
- R2: footprint Resistors_SMD:R_2010_HandSoldering -> Resistors_SMD:R_2512_HandSoldering
Connections:
- net 9VAC1+: now also J2.5 (Pin_5), J2.6 (Pin_6), J2.7 (Pin_7), J2.8 (Pin_8); no longer J2.1 (Pin_1), J2.2 (Pin_2), J2.3 (Pin_3), J2.4 (Pin_4)
- net 9VAC1-: now also J2.1 (Pin_1), J2.2 (Pin_2), J2.3 (Pin_3), J2.4 (Pin_4); no longer J2.5 (Pin_5), J2.6 (Pin_6), J2.7 (Pin_7), J2.8 (Pin_8)
- net VIN+: now also J1.5 (Pin_5), J1.6 (Pin_6), J1.7 (Pin_7), J1.8 (Pin_8); no longer J1.1 (Pin_1), J1.2 (Pin_2), J1.3 (Pin_3), J1.4 (Pin_4)
- net VIN-: now also J1.1 (Pin_1), J1.2 (Pin_2), J1.3 (Pin_3), J1.4 (Pin_4); no longer J1.5 (Pin_5), J1.6 (Pin_6), J1.7 (Pin_7), J1.8 (Pin_8)
Other:
- note added: "2017-07-23"
Changed lines of the file:
@@
 F 0 "R2" V 1280 1550 50  0000 C CNN
 F 1 "0R1" V 1200 1550 50  0000 C CNN
-F 2 "Resistors_SMD:R_2010_HandSoldering" V 1130 1550 50  0001 C CNN
+F 2 "Resistors_SMD:R_2512_HandSoldering" V 1130 1550 50  0001 C CNN
 F 3 "" H 1200 1550 50  0001 C CNN
 	1    1200 1550
@@
 F 0 "C1" H 6375 2350 50  0000 L CNN
 F 1 "220u" H 6375 2150 50  0000 L CNN
-F 2 "Capacitors_SMD:C_1210_HandSoldering" H 6388 2100 50  0001 C CNN
+F 2 "Capacitors_Tantalum_SMD:CP_Tantalum_Case-X_EIA-7343-43_Reflow" H 6388 2100 50  0001 C CNN
 F 3 "" H 6350 2250 50  0001 C CNN
 	1    6350 2250
@@
 L Conn_01x08_Female J1
 U 1 1 5B426E14
-P 1300 950
-F 0 "J1" H 1300 1350 50  0000 C CNN
-F 1 "Conn_01x08_Female" H 1300 450 50  0000 C CNN
-F 2 "Pin_Headers:Pin_Header_Straight_1x08_Pitch2.54mm" H 1300 950 50  0001 C CNN
-F 3 "" H 1300 950 50  0001 C CNN
-	1    1300 950
-	0    -1   -1   0
+P 1400 950
+F 0 "J1" H 1400 1350 50  0000 C CNN
+F 1 "Conn_01x08_Female" H 1400 450 50  0000 C CNN
+F 2 "Pin_Headers:Pin_Header_Straight_1x08_Pitch2.54mm" H 1400 950 50  0001 C CNN
+F 3 "" H 1400 950 50  0001 C CNN
+	1    1400 950
+	0    1    -1   0
 $EndComp
 $Comp
 L Conn_01x08_Female J2
 U 1 1 5B427C9D
-P 2550 6900
-F 0 "J2" H 2550 7300 50  0000 C CNN
-F 1 "Conn_01x08_Female" H 2550 6400 50  0000 C CNN
-F 2 "Pin_Headers:Pin_Header_Straight_1x08_Pitch2.54mm" H 2550 6900 50  0001 C CNN
-F 3 "" H 2550 6900 50  0001 C CNN
-	1    2550 6900
-	0    -1   1    0
+P 2650 6900
+F 0 "J2" H 2650 7300 50  0000 C CNN
+F 1 "Conn_01x08_Female" H 2650 6400 50  0000 C CNN
+F 2 "Pin_Headers:Pin_Header_Straight_1x08_Pitch2.54mm" H 2650 6900 50  0001 C CNN
+F 3 "" H 2650 6900 50  0001 C CNN
+	1    2650 6900
+	0    1    1    0
 $EndComp
 $Comp
@@
 Text Label 8100 1150 0    60   ~ 0
 FILTER
+Text Notes 8200 7650 0    60   ~ 0
+2017-07-23
 $EndSCHEMATC
