File: addon board/C64Saver2-addon.sch (KiCad schematic (older format))
At the start: 38 parts, among them CON1 AVR-ISP-6, J1 Conn_01x08_Female, J2 Conn_01x08_Female, J3 OLED_128x32_Conn_01x04_Male, J4 Conn_01x04_Female, SW1 SW_Push, U1 INA219xIDR-SOIC, U2 ISO1541D, U3 ATTINY85-20SU, U4 TLP291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

Commit message: Change: ATtiny footprint, ADC used with reset input
Parts:
- added R13: 10k, Resistors_SMD:R_0603_HandSoldering, symbol R_Small
- added R14: 1k, Resistors_SMD:R_0603_HandSoldering, symbol R_Small
- U3: footprint Housings_SOIC:SOIC-8_3.9x4.9mm_Pitch1.27mm -> Housings_SOIC:SOIJ-8_5.3x5.3mm_Pitch1.27mm
Connections:
- net #OVERVOLTAGE: now also R13.1, R14.1; no longer U5.4
- net +5V: now also R14.2
- new net: R13.2, U5.4
Other:
- note added: "1.1"
- note added: "2018-09-09"
- note removed: "1.0"
- note removed: "2017-07-23"
Changed lines of the file:
@@
 	0    1    1    0
 $EndComp
-Text Label 5300 5800 0    60   ~ 0
+Text Label 6250 5800 0    60   ~ 0
 #OVERVOLTAGE
 $Comp
@@
 $EndComp
 Text Notes 10650 7650 0    60   ~ 0
-1.0
+1.1
 Text Label 5750 2600 0    60   ~ 0
 9VAC2
@@
 F 0 "U3" H 8300 5700 50  0000 C CNN
 F 1 "ATTINY85-20SU" H 10450 4900 50  0000 C CNN
-F 2 "Housings_SOIC:SOIC-8_3.9x4.9mm_Pitch1.27mm" H 10400 5300 50  0001 C CIN
+F 2 "Housings_SOIC:SOIJ-8_5.3x5.3mm_Pitch1.27mm" H 10400 5300 50  0001 C CIN
 F 3 "" H 9450 5300 50  0001 C CNN
 	1    9450 5300
@@
 	5150 6000 5200 6000
 Wire Wire Line
-	5150 5800 7000 5800
-Wire Wire Line
 	2950 5400 2950 5300
 Connection ~ 2950 4900
@@
 	3600 6400 3600 6700
 Wire Wire Line
-	8100 5450 7300 5450
-Wire Wire Line
-	7300 5450 6050 5050
-Wire Wire Line
-	6050 5050 6000 5050
+	7000 5450 8100 5450
+Wire Wire Line
+	6000 5050 7000 5050
 Wire Wire Line
 	7900 5150 8100 5150
@@
 FILTER
 Text Notes 8200 7650 0    60   ~ 0
-2017-07-23
+2018-09-09
+Wire Wire Line
+	7000 5050 7000 5450
+$Comp
+L R_Small R13
+U 1 1 5B9332FC
+P 5800 5800
+F 0 "R13" V 5750 5600 50  0000 L CNN
+F 1 "10k" V 5800 5750 39  0000 L CNN
+F 2 "Resistors_SMD:R_0603_HandSoldering" H 5800 5800 50  0001 C CNN
+F 3 "" H 5800 5800 50  0001 C CNN
+	1    5800 5800
+	0    1    1    0
+$EndComp
+$Comp
+L R_Small R14
+U 1 1 5B9333B5
+P 6000 5650
+F 0 "R14" V 5900 5550 50  0000 L CNN
+F 1 "1k" V 6000 5600 39  0000 L CNN
+F 2 "Resistors_SMD:R_0603_HandSoldering" H 6000 5650 50  0001 C CNN
+F 3 "" H 6000 5650 50  0001 C CNN
+	1    6000 5650
+	-1   0    0    1
+$EndComp
+$Comp
+L +5V #PWR026
+U 1 1 5B93348B
+P 6000 5550
+F 0 "#PWR026" H 6000 5400 50  0001 C CNN
+F 1 "+5V" H 6000 5690 50  0000 C CNN
+F 2 "" H 6000 5550 50  0001 C CNN
+F 3 "" H 6000 5550 50  0001 C CNN
+	1    6000 5550
+	1    0    0    -1
+$EndComp
+Wire Wire Line
+	7000 5800 5900 5800
+Wire Wire Line
+	5700 5800 5150 5800
+Wire Wire Line
+	6000 5750 6000 5800
+Connection ~ 6000 5800
 $EndSCHEMATC

Commit message: Addon board ready for new release #9
Parts:
- U7, U8: value MCP1700-5002E_SOT23 -> MCP1703
Other:
- note added: "2018-09-23"
- note removed: "2018-09-09"
Changed lines of the file:
@@
 P 2050 2950
 F 0 "U8" H 1900 3075 50  0000 C CNN
-F 1 "MCP1700-5002E_SOT23" H 1850 3150 50  0000 L CNN
+F 1 "MCP1703" H 1850 3150 50  0000 L CNN
 F 2 "TO_SOT_Packages_SMD:SOT-23" H 2050 3175 50  0001 C CNN
 F 3 "" H 2050 2950 50  0001 C CNN
@@
 P 7100 1950
 F 0 "U7" H 6950 2075 50  0000 C CNN
-F 1 "MCP1700-5002E_SOT23" H 6900 2150 50  0000 L CNN
+F 1 "MCP1703" H 6900 2150 50  0000 L CNN
 F 2 "TO_SOT_Packages_SMD:SOT-23" H 7100 2175 50  0001 C CNN
 F 3 "" H 7100 1950 50  0001 C CNN
@@
 FILTER
 Text Notes 8200 7650 0    60   ~ 0
-2018-09-09
+2018-09-23
 Wire Wire Line
 	7000 5050 7000 5450

Commit message: addonboard: 5V moved to VIN+, and fixed SDA2 and SCL2. #16 #17
Connections:
- net SCL2: now also U1.4 (SCL); no longer R9.1, U1.3 (SDA)
- net SDA2: now also U1.3 (SDA); no longer R7.1, U1.4 (SCL)
- net VIN+: now also C6.2, U8.3 (VI)
- net VIN-: no longer C6.2, U8.3 (VI)
Other:
- note added: "1.2"
- note added: "2018-11-04"
- note removed: "1.1"
- note removed: "2018-09-23"
Changed lines of the file:
@@
 $EndComp
 Text Notes 10650 7650 0    60   ~ 0
-1.1
+1.2
 Text Label 5750 2600 0    60   ~ 0
 9VAC2
@@
 Connection ~ 1350 4550
 Wire Wire Line
-	2800 4100 4400 4100
-Wire Wire Line
-	2800 4200 3200 4200
-Wire Wire Line
 	2950 4800 2950 5100
 Wire Wire Line
@@
 	3300 5750 2250 5750
 Wire Wire Line
-	3200 4300 4400 4300
-Wire Wire Line
-	9100 900  8100 900
+	8100 900  9100 900
 Wire Wire Line
 	8900 4200 8900 1000
@@
 Wire Wire Line
 	6050 3700 6050 3750
-Wire Wire Line
-	3200 4200 3200 4300
-Wire Wire Line
-	2900 4000 2900 4100
-Connection ~ 2900 4100
-Wire Wire Line
-	3100 4000 3100 4200
-Connection ~ 3100 4200
 Wire Wire Line
 	2900 3800 2900 3750
@@
 Connection ~ 2050 3350
 Wire Wire Line
-	1050 2950 1750 2950
+	1000 2950 1750 2950
 Connection ~ 1700 2950
 Wire Wire Line
@@
 Wire Wire Line
 	1700 2950 1700 3000
-Connection ~ 1050 2950
 Connection ~ 2750 3600
 Wire Wire Line
@@
 	7900 4300 9900 4300
 Wire Wire Line
-	8100 5250 7400 5250
-Wire Wire Line
-	7400 5250 7400 4100
+	7400 5250 8100 5250
+Wire Wire Line
+	7400 4100 7400 5250
 Wire Wire Line
 	7500 5050 8100 5050
@@
 FILTER
 Text Notes 8200 7650 0    60   ~ 0
-2018-09-23
+2018-11-04
 Wire Wire Line
 	7000 5050 7000 5450
@@
 $EndComp
 Wire Wire Line
-	7000 5800 5900 5800
+	5900 5800 7000 5800
 Wire Wire Line
 	5700 5800 5150 5800
@@
 	6000 5750 6000 5800
 Connection ~ 6000 5800
+Wire Wire Line
+	4400 4100 4150 4100
+Wire Wire Line
+	2800 4100 3100 4100
+Wire Wire Line
+	4150 4100 4150 4200
+Wire Wire Line
+	4150 4200 2800 4200
+Wire Wire Line
+	3100 4100 3100 4300
+Wire Wire Line
+	3100 4300 4400 4300
+Connection ~ 1000 2950
 $EndSCHEMATC

Commit message: 4k7 pullups + readme
Parts:
- R10, R11, R7, R9: value 560 -> 4k7
Connections:
- net SCL2: now also R9.1
- net SDA2: now also R7.1
Changed lines of the file:
@@
 P 6050 3850
 F 0 "R10" V 5950 3750 50  0000 L CNN
-F 1 "560" V 6050 3800 39  0000 L CNN
+F 1 "4k7" V 6050 3800 39  0000 L CNN
 F 2 "Resistors_SMD:R_0603_HandSoldering" H 6050 3850 50  0001 C CNN
 F 3 "" H 6050 3850 50  0001 C CNN
@@
 P 6250 3850
 F 0 "R11" V 6150 3750 50  0000 L CNN
-F 1 "560" V 6250 3800 39  0000 L CNN
+F 1 "4k7" V 6250 3800 39  0000 L CNN
 F 2 "Resistors_SMD:R_0603_HandSoldering" H 6250 3850 50  0001 C CNN
 F 3 "" H 6250 3850 50  0001 C CNN
@@
 P 2900 3900
 F 0 "R7" V 2800 3800 50  0000 L CNN
-F 1 "560" V 2900 3850 39  0000 L CNN
+F 1 "4k7" V 2900 3850 39  0000 L CNN
 F 2 "Resistors_SMD:R_0603_HandSoldering" H 2900 3900 50  0001 C CNN
 F 3 "" H 2900 3900 50  0001 C CNN
@@
 P 3100 3900
 F 0 "R9" V 3000 3800 50  0000 L CNN
-F 1 "560" V 3100 3850 39  0000 L CNN
+F 1 "4k7" V 3100 3850 39  0000 L CNN
 F 2 "Resistors_SMD:R_0603_HandSoldering" H 3100 3900 50  0001 C CNN
 F 3 "" H 3100 3900 50  0001 C CNN
@@
 	4150 4200 2800 4200
 Wire Wire Line
-	3100 4100 3100 4300
+	3100 4000 3100 4300
 Wire Wire Line
 	3100 4300 4400 4300
 Connection ~ 1000 2950
+Wire Wire Line
+	2900 4000 2900 4200
+Connection ~ 2900 4200
+Connection ~ 3100 4100
 $EndSCHEMATC

Commit message: Swapped HOLD_ with SENSE_VAC #18
Parts:
- C1: value 220u -> 100u Case-X
- D1: value D -> Dotec SL1G
Connections:
- net HOLD_: now also CON1.1, U3.6 (PB1(MISO/DO/AIN1/OC0B/OC1A/PCINT1)); no longer U3.3 (PB4(XTAL2/CLKO/OC1B/ADC2/PCINT4))
- net SENSE_VAC: now also U3.3 (PB4(XTAL2/CLKO/OC1B/ADC2/PCINT4)); no longer CON1.1, U3.6 (PB1(MISO/DO/AIN1/OC0B/OC1A/PCINT1))
Other:
- note added: "2018-11-11"
- note removed: "2018-11-04"
Changed lines of the file:
@@
 P 5900 1950
 F 0 "D1" H 5900 2050 50  0000 C CNN
-F 1 "D" H 5900 1850 50  0000 C CNN
+F 1 "Dotec SL1G" H 5900 1850 50  0000 C CNN
 F 2 "Diodes_SMD:D_SOD-123" H 5900 1950 50  0001 C CNN
 F 3 "" H 5900 1950 50  0001 C CNN
@@
 U 1 1 5B2D5A0C
 P 6350 2250
-F 0 "C1" H 6375 2350 50  0000 L CNN
-F 1 "220u" H 6375 2150 50  0000 L CNN
+F 0 "C1" H 6100 2250 50  0000 L CNN
+F 1 "100u Case-X" H 5750 2350 50  0000 L CNN
 F 2 "Capacitors_Tantalum_SMD:CP_Tantalum_Case-X_EIA-7343-43_Reflow" H 6388 2100 50  0001 C CNN
 F 3 "" H 6350 2250 50  0001 C CNN
@@
 	1    0    0    -1
 $EndComp
-Text Label 7350 5450 0    60   ~ 0
+Text Label 6300 5050 0    60   ~ 0
 HOLD_
 $Comp
@@
 	3600 6400 3600 6700
 Wire Wire Line
-	7000 5450 8100 5450
-Wire Wire Line
-	6000 5050 7000 5050
-Wire Wire Line
-	7900 5150 8100 5150
-Wire Wire Line
-	7900 5150 7900 4300
+	6000 5050 7100 5050
 Wire Wire Line
 	7800 4200 7800 5350
@@
 Wire Wire Line
 	8000 5850 8000 5150
-Connection ~ 8000 5150
 Wire Wire Line
 	7550 6250 7400 6250
@@
 FILTER
 Text Notes 8200 7650 0    60   ~ 0
-2018-11-04
-Wire Wire Line
-	7000 5050 7000 5450
+2018-11-11
 $Comp
 L R_Small R13
@@
 Connection ~ 2900 4200
 Connection ~ 3100 4100
+Wire Wire Line
+	7100 5150 8100 5150
+Wire Wire Line
+	7100 5050 7100 5150
+Connection ~ 8000 5150
+Wire Wire Line
+	8100 5450 7900 5450
+Wire Wire Line
+	7900 5450 7900 4300
 $EndSCHEMATC
