File: addon board/C64Saver2-addon.sch (KiCad schematic (older format))
At the start: 40 parts, among them CON1 AVR-ISP-6, J1 Conn_01x08_Female, J2 Conn_01x08_Female, J3 OLED_128x32_Conn_01x04_Male, J4 Conn_01x04_Female, SW1 SW_Push, U1 INA219xIDR-SOIC, U2 ISO1541D, U3 ATTINY85-20SU, U4 TLP291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

Commit message: Addon Board 1.3 (2019-05-24)
  - Changed optocoupler footprint to more common SOIC-4_4.55x2.6mm_P1.27mm
  - Larger 5V regulator on 9vac side for less heat
  - replaced 100uF tantalum with 3x 47uF 1206 MLCC
  - kicad 5.1.0 project
Parts:
- removed C1: 100u Case-X, Capacitors_Tantalum_SMD:CP_Tantalum_Case-X_EIA-7343-43_Reflow, symbol Device:C
- added C1, C12, C13: 47uF, Capacitor_SMD:C_1206_3216Metric, symbol Device:C_Small
- U4, U5: value TLP291 -> ACPL-217-50DE; footprint Housings_SOIC:SO-4_7.6x3.6mm_Pitch2.54mm -> Package_SO:SOIC-4_4.55x2.6mm_P1.27mm
- U7: footprint TO_SOT_Packages_SMD:SOT-23 -> Package_TO_SOT_SMD:SOT-223-3_TabPin2
Connections:
- net GND: now also C1.2, C12.2, C13.2
- net at D1.1 (K), U7.3 (VI): now also C1.1, C12.1, C13.1
Other:
- note added: "GRM31CR61E476ME44K"
- note removed: "1.2"
- note removed: "2018-11-11"
- moved on the sheet: D1
Changed lines of the file:
@@
 encoding utf-8
 Sheet 1 1
-Title ""
-Date ""
-Rev ""
-Comp ""
+Title "C64 Saver 2 Addon Board"
+Date "2019-05-24"
+Rev "1.3"
+Comp "BWACK"
 Comment1 ""
 Comment2 ""
@@
 L Device:D D1
 U 1 1 5B21A217
-P 5900 1950
-F 0 "D1" H 5900 2050 50  0000 C CNN
-F 1 "Dotec SL1G" H 5900 1850 50  0000 C CNN
-F 2 "Diodes_SMD:D_SOD-123" H 5900 1950 50  0001 C CNN
-F 3 "" H 5900 1950 50  0001 C CNN
-	1    5900 1950
+P 5700 1950
+F 0 "D1" H 5700 2050 50  0000 C CNN
+F 1 "Dotec SL1G" H 5700 1850 50  0000 C CNN
+F 2 "Diodes_SMD:D_SOD-123" H 5700 1950 50  0001 C CNN
+F 3 "" H 5700 1950 50  0001 C CNN
+	1    5700 1950
 	-1   0    0    -1
 $EndComp
@@
 Text Label 5750 1150 0    60   ~ 0
 9VAC1-
-$Comp
-L Device:C C1
-U 1 1 5B2D5A0C
-P 6350 2250
-F 0 "C1" H 6100 2250 50  0000 L CNN
-F 1 "100u Case-X" H 5750 2350 50  0000 L CNN
-F 2 "Capacitors_Tantalum_SMD:CP_Tantalum_Case-X_EIA-7343-43_Reflow" H 6388 2100 50  0001 C CNN
-F 3 "" H 6350 2250 50  0001 C CNN
-	1    6350 2250
-	-1   0    0    1
-$EndComp
-Text Notes 10650 7650 0    60   ~ 0
-1.2
-Text Label 5750 2600 0    60   ~ 0
+Text Label 5500 2600 0    60   ~ 0
 9VAC2
 $Comp
@@
 P 4850 5150
 F 0 "U4" H 4650 5350 50  0000 L CNN
-F 1 "TLP291" H 4850 5350 50  0000 L CNN
-F 2 "Housings_SOIC:SO-4_7.6x3.6mm_Pitch2.54mm" H 4650 4950 50  0001 L CIN
+F 1 "ACPL-217-50DE" H 4850 5350 50  0000 L CNN
+F 2 "Package_SO:SOIC-4_4.55x2.6mm_P1.27mm" H 4650 4950 50  0001 L CIN
 F 3 "" H 4850 5150 50  0001 L CNN
 	1    4850 5150
@@
 P 4850 5900
 F 0 "U5" H 4650 6100 50  0000 L CNN
-F 1 "TLP291" H 4850 6100 50  0000 L CNN
-F 2 "Housings_SOIC:SO-4_7.6x3.6mm_Pitch2.54mm" H 4650 5700 50  0001 L CIN
+F 1 "ACPL-217-50DE" H 4850 6100 50  0000 L CNN
+F 2 "Package_SO:SOIC-4_4.55x2.6mm_P1.27mm" H 4650 5700 50  0001 L CIN
 F 3 "" H 4850 5900 50  0001 L CNN
 	1    4850 5900
@@
 F 0 "U8" H 1900 3075 50  0000 C CNN
 F 1 "MCP1703" H 1850 3150 50  0000 L CNN
-F 2 "TO_SOT_Packages_SMD:SOT-23" H 2050 3175 50  0001 C CNN
+F 2 "TO_SOT_Packages_SMD:SOT-23" H 2200 3250 50  0000 C CNN
 F 3 "" H 2050 2950 50  0001 C CNN
 	1    2050 2950
@@
 F 0 "U7" H 6950 2075 50  0000 C CNN
 F 1 "MCP1703" H 6900 2150 50  0000 L CNN
-F 2 "TO_SOT_Packages_SMD:SOT-23" H 7100 2175 50  0001 C CNN
+F 2 "Package_TO_SOT_SMD:SOT-223-3_TabPin2" H 7650 2200 50  0000 C CNN
 F 3 "" H 7100 1950 50  0001 C CNN
 	1    7100 1950
@@
 	3500 5950 3500 2600
 Wire Wire Line
-	3500 2600 6350 2600
-Wire Wire Line
-	5550 1950 5750 1950
-Wire Wire Line
-	6050 1950 6350 1950
-Wire Wire Line
-	6350 1950 6350 2100
-Wire Wire Line
-	6350 2400 6350 2600
-Connection ~ 6350 2600
-Connection ~ 6350 1950
+	3500 2600 6000 2600
+Wire Wire Line
+	5850 1950 6000 1950
 Wire Wire Line
 	7100 2250 7100 2600
@@
 Text Label 8100 1150 0    60   ~ 0
 FILTER
-Text Notes 8200 7650 0    60   ~ 0
-2018-11-11
 $Comp
 L Device:R_Small R13
@@
 	6950 1150 7000 1150
 Wire Wire Line
-	6350 2600 7100 2600
-Wire Wire Line
-	6350 1950 6800 1950
-Wire Wire Line
 	7100 2600 7550 2600
 Wire Wire Line
@@
 Wire Wire Line
 	8000 5150 8100 5150
+$Comp
+L Device:C_Small C1
+U 1 1 5CE4F594
+P 6000 2250
+F 0 "C1" H 6050 2400 50  0000 L CNN
+F 1 "47uF" H 6050 2300 50  0000 L CNN
+F 2 "Capacitor_SMD:C_1206_3216Metric" H 6000 2250 50  0001 C CNN
+F 3 "~" H 6000 2250 50  0001 C CNN
+	1    6000 2250
+	1    0    0    -1
+$EndComp
+$Comp
+L Device:C_Small C12
+U 1 1 5CE514C4
+P 6300 2250
+F 0 "C12" H 6350 2400 50  0000 L CNN
+F 1 "47uF" H 6350 2300 50  0000 L CNN
+F 2 "Capacitor_SMD:C_1206_3216Metric" H 6300 2250 50  0001 C CNN
+F 3 "~" H 6300 2250 50  0001 C CNN
+	1    6300 2250
+	1    0    0    -1
+$EndComp
+$Comp
+L Device:C_Small C13
+U 1 1 5CE5183F
+P 6600 2250
+F 0 "C13" H 6650 2400 50  0000 L CNN
+F 1 "47uF" H 6650 2300 50  0000 L CNN
+F 2 "Capacitor_SMD:C_1206_3216Metric" H 6600 2250 50  0001 C CNN
+F 3 "~" H 6600 2250 50  0001 C CNN
+	1    6600 2250
+	1    0    0    -1
+$EndComp
+Wire Wire Line
+	6000 2150 6000 1950
+Connection ~ 6000 1950
+Wire Wire Line
+	6000 1950 6300 1950
+Wire Wire Line
+	6000 2350 6000 2600
+Connection ~ 6000 2600
+Wire Wire Line
+	6000 2600 6300 2600
+Wire Wire Line
+	6300 2150 6300 1950
+Connection ~ 6300 1950
+Wire Wire Line
+	6300 2350 6300 2600
+Connection ~ 6300 2600
+Wire Wire Line
+	6300 2600 6600 2600
+Wire Wire Line
+	6300 1950 6600 1950
+Wire Wire Line
+	6600 2150 6600 1950
+Connection ~ 6600 1950
+Wire Wire Line
+	6600 1950 6800 1950
+Wire Wire Line
+	6600 2350 6600 2600
+Connection ~ 6600 2600
+Wire Wire Line
+	6600 2600 7100 2600
+Text Notes 5800 2400 0    60   ~ 0
+GRM31CR61E476ME44K
 $EndSCHEMATC

Commit message: kicad 5.1.0 -> 5.1.2
Parts:
- R6: footprint Resistors_SMD:R_0603_HandSoldering -> Resistor_SMD:R_0603_1608Metric_Pad1.05x0.95mm_HandSolder
- U1, U2, U6: footprint SMD_Packages:SOIC-8-N -> Package_SO:SOIC-8_3.9x4.9mm_P1.27mm
- U3: footprint Housings_SOIC:SOIJ-8_5.3x5.3mm_Pitch1.27mm -> Package_SO:SOIJ-8_5.3x5.3mm_P1.27mm
Changed lines of the file:
@@
 F 0 "U1" H 1650 4950 50  0000 L CNN
 F 1 "INA219xIDR-SOIC" H 2150 4950 50  0000 L CNN
-F 2 "SMD_Packages:SOIC-8-N" H 2850 3900 50  0001 C CNN
+F 2 "Package_SO:SOIC-8_3.9x4.9mm_P1.27mm" H 2850 3900 50  0001 C CNN
 F 3 "" H 2000 4100 50  0000 C CNN
 	1    1900 4450
@@
 F 0 "U2" H 4500 4600 50  0000 L CNN
 F 1 "ISO1541D" H 4750 4600 50  0000 L CNN
-F 2 "SMD_Packages:SOIC-8-N" H 4950 3800 50  0001 C CIN
+F 2 "Package_SO:SOIC-8_3.9x4.9mm_P1.27mm" H 4950 3800 50  0001 C CIN
 F 3 "" H 4850 4200 50  0001 C CNN
 	1    4850 4200
@@
 F 0 "R6" H 9400 4350 50  0000 L CNN
 F 1 "470k" H 9400 4450 39  0000 L CNN
-F 2 "Resistors_SMD:R_0603_HandSoldering" H 9600 4450 50  0001 C CNN
+F 2 "Resistor_SMD:R_0603_1608Metric_Pad1.05x0.95mm_HandSolder" H 9600 4450 50  0001 C CNN
 F 3 "" H 9600 4450 50  0001 C CNN
 	1    9600 4450
@@
 F 0 "U6" H 7550 1350 60  0000 C CNN
 F 1 "ACS712" H 7550 700 60  0000 C CNN
-F 2 "SMD_Packages:SOIC-8-N" H 7550 1050 60  0001 C CNN
+F 2 "Package_SO:SOIC-8_3.9x4.9mm_P1.27mm" H 7550 1050 60  0001 C CNN
 F 3 "" H 7550 1050 60  0001 C CNN
 	1    7550 1050
@@
 F 0 "U3" H 8300 5700 50  0000 C CNN
 F 1 "ATTINY85-20SU" H 10450 4900 50  0000 C CNN
-F 2 "Housings_SOIC:SOIJ-8_5.3x5.3mm_Pitch1.27mm" H 10400 5300 50  0001 C CIN
+F 2 "Package_SO:SOIJ-8_5.3x5.3mm_P1.27mm" H 10400 5300 50  0001 C CIN
 F 3 "" H 9450 5300 50  0001 C CNN
 	1    9450 5300
