File: C64 Saver 2/C64Saver2.kicad_pcb (KiCad board)
At the start: 2 copper layers, 43.9 x 28.8 mm, 22 parts, among them J1 Conn_01x04, J2 Conn_01x08, J4 Conn_01x08, J5 Conn_01x04, J6 Conn_01x04, Q1 2N7000, Q2 IRFR5305

Commit message: Added IN/OUT to bottom silkscreen. upped project to Kicad 5.1.2
Parts:
- removed REF**: HAMMOND_1551G, HAMMOND:HAMMOND_1551G
Other:
- board text added: "OUT"

Commit message: C64 Saver 2.5 ready for prototype
Parts:
- removed D3: 6V8, Diodes_THT:D_DO-35_SOD27_P7.62mm_Horizontal
- added LED1: LED_RED_3mm, LED_THT:LED_D3.0mm, F.Cu at (153.7, 99.1)
- added LED2: LED_GREEN_3mm, LED_THT:LED_D3.0mm, F.Cu at (156.2, 103.6)
- added R10: 3k3, Resistor_SMD:R_0805_2012Metric_Pad1.15x1.40mm_HandSolder, F.Cu at (161.9, 101.6)
- added R11: 3k3, Resistor_SMD:R_0805_2012Metric_Pad1.15x1.40mm_HandSolder, F.Cu at (159.4, 101.6)
- added R9: 3k3, Resistor_SMD:R_0805_2012Metric_Pad1.15x1.40mm_HandSolder, F.Cu at (150.1, 99.7)
- added U1: TL431DBZ, Package_TO_SOT_SMD:SOT-23, F.Cu at (169.5, 91.4)
- C1: footprint Capacitors_THT:CP_Radial_D6.3mm_P2.50mm -> Capacitor_SMD:CP_Elec_6.3x5.4
- D1: value TL431LP -> BZY55B6V8; footprint TO_SOT_Packages_THT:TO-92_Inline_Narrow_Oval -> Diode_SMD:D_0805_2012Metric_Pad1.15x1.40mm_HandSolder
- D2: value 6V8 -> BZY55B6V8; footprint Diodes_THT:D_DO-35_SOD27_P7.62mm_Horizontal -> Diode_SMD:D_0805_2012Metric_Pad1.15x1.40mm_HandSolder
- Q1: value 2N7000 -> 2N7002; footprint TO_SOT_Packages_THT:TO-92_Inline_Wide -> Package_TO_SOT_SMD:SOT-23
- R1, R2, R3, R4, R5, R6, R7, R8: footprint Resistors_THT:R_Axial_DIN0204_L3.6mm_D1.6mm_P5.08mm_Horizontal -> Resistor_SMD:R_0805_2012Metric_Pad1.15x1.40mm_HandSolder
- moved R8 19.3 mm to (172.7, 96.5), turned to 270 degrees
- moved R7 17.1 mm to (172.7, 91.4)
- moved D2 16.3 mm to (161.3, 91.4), turned to 270 degrees
- moved R4 11.5 mm to (165.1, 101.6)
- moved R1 10.2 mm to (163.8, 91.4)
- moved D1 9.43 mm to (175.3, 96.5)
- moved Q1 8.32 mm to (169.5, 96.5), turned to 0 degrees
- moved R2 8.13 mm to (166.4, 96.5)
- moved R5 6.35 mm to (163.8, 96.5)
- moved R6 6.35 mm to (161.3, 96.5), turned to 90 degrees
- moved C1 3.12 mm to (171.4, 102.2), turned to 0 degrees
- moved R3 2.81 mm to (166.4, 91.4)
Connections:
- C1 pad 1: /VCC1- -> /VCC1+
- D1 pad 1: /SENSE -> /NGATE
- D2 pad 1: /NGATE -> /VCC1-
- D2 pad 2: GND -> PGATE
- Q1 pad 1: GND -> /NGATE
- Q1 pad 2: /NGATE -> GND
- R3 pad 2: Net-(D1-Pad3) -> Net-(R3-Pad2)
- R7 pad 1: Net-(D1-Pad3) -> Net-(R3-Pad2)
Routing:
- net PGATE: track 56.4 -> 19.9 mm
- net GND: track 17.1 -> 48.6 mm, vias 0 -> 4
- net Net-(D1-Pad3): track 17.1 -> 0.00 mm
- net /VCC1+: track 17.5 -> 34.3 mm
- net /VCC1-: track 51.9 -> 38.3 mm, vias 1 -> 0
- net /5V_SAFE: track 0.00 -> 11.0 mm
- net OVERVOLTAGE: track 21.3 -> 32.0 mm, vias 1 -> 0
- net /SENSE: track 22.4 -> 13.6 mm
- net Net-(R3-Pad2): track 0.00 -> 7.17 mm
- net /9VAC1: track 29.9 -> 23.7 mm
- net /NGATE: track 11.6 -> 16.1 mm
- net Net-(LED1-Pad1): track 0.00 -> 4.24 mm
- net Net-(LED2-Pad1): track 0.00 -> 3.59 mm
- net /9VAC2: track 44.1 -> 44.9 mm
Other:
- board text added: "C64 Saver 2.5 BWACK 2020"
- board text removed: "C64 Saver Rev 2.4 BWACK 2018"
