File: C64 Saver 2/C64Saver2.sch (KiCad schematic (older format))
At the start: 21 parts, among them J1 Conn_01x04, J2 Conn_01x08, J4 Conn_01x08, J5 Conn_01x04, J6 Conn_01x04, Q1 2N7000, Q2 IRFR5305

Commit message: C64 Saver 2.5 ready for prototype
Parts:
- removed D1: TL431LP, TO_SOT_Packages_THT:TO-92_Inline_Narrow_Oval, symbol C64Saver2-rescue:TL431LP
- removed D2, D3: 6V8, Diodes_THT:D_DO-35_SOD27_P7.62mm_Horizontal, symbol C64Saver2-rescue:D_Zener_Small
- removed Q1: 2N7000, TO_SOT_Packages_THT:TO-92_Inline_Wide, symbol C64Saver2-rescue:2N7000
- added D1, D2: BZY55B6V8, Diode_SMD:D_0805_2012Metric_Pad1.15x1.40mm_HandSolder, symbol Device:D_Zener_ALT
- added LED1: LED_RED_3mm, LED_THT:LED_D3.0mm, symbol Device:LED_ALT
- added LED2: LED_GREEN_3mm, LED_THT:LED_D3.0mm, symbol Device:LED_ALT
- added Q1: 2N7002, Package_TO_SOT_SMD:SOT-23, symbol Transistor_FET:2N7002
- added R10, R11, R9: 3k3, Resistor_SMD:R_0805_2012Metric_Pad1.15x1.40mm_HandSolder, symbol C64Saver2-rescue:R
- added U1: TL431DBZ, Package_TO_SOT_SMD:SOT-23, symbol Reference_Voltage:TL431DBZ
- C1: footprint Capacitors_THT:CP_Radial_D6.3mm_P2.50mm -> Capacitor_SMD:CP_Elec_6.3x5.4
- R1, R2, R3, R4, R5, R6, R7, R8: footprint Resistors_THT:R_Axial_DIN0204_L3.6mm_D1.6mm_P5.08mm_Horizontal -> Resistor_SMD:R_0805_2012Metric_Pad1.15x1.40mm_HandSolder
Connections:
- net 5V_SAFE: now also LED2.2 (A), R10.2, R9.1
- net GND: now also D1.2 (A), Q1.2 (S), R10.1, R11.1, U1.3 (A)
- net NGATE: now also D1.1 (K), Q1.1 (G)
- net OVERVOLTAGE: now also Q1.3 (D)
- net PGATE: now also D2.2 (A)
- net SENSE: now also U1.2 (REF)
- net VCC1+: now also C1.1
- net VCC1-: now also D2.1 (K), LED1.2 (A); no longer C1.1
- net at R3.2, R7.1: now also U1.1 (K)
- new net: LED1.1 (K), R9.2
- new net: LED2.1 (K), R11.2
Other:
- note removed: "2.4"
- note removed: "2018-09-23"
- note removed: "C64 Saver"
- moved on the sheet: C1, R5
