File: addon board 1.4/C64Saver2-addon.kicad_pcb (KiCad board)
At the start: 2 copper layers, 43.9 x 29 mm, 43 parts, among them CON1 AVR-ISP-6, J1 Conn_01x08_Female, J2 Conn_01x08_Female, J3 OLED_128x32_Conn_01x04_Male, J4 Conn_01x04_Female, SW1 SW_Push, U1 INA219xIDR-SOIC, U2 ISO1541D, U3 ATTINY85-20SU, U4 ACPL-217-50DE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

Commit message: Added ibom for addon board, and put the elfa+RS components into the parts/ibom
Parts:
- removed REF**: HAMMOND_1551G, HAMMOND:HAMMOND_1551G
- R10, R11, R7, R8, R9: value 4k7 -> 4K7
- R13: value 10k -> 10K
- R14: value 1k -> 1K
- R5, R6: value 470k -> 470K
