File: addon board 1.4/C64Saver2-addon.kicad_sch (KiCad schematic)
At the start: 42 parts, among them CON1 AVR-ISP-6, J1 Conn_01x08_Female, J2 Conn_01x08_Female, J3 OLED_128x32_Conn_01x04_Male, J4 Conn_01x04_Female, SW1 SW_Push, U1 INA219xIDR-SOIC, U2 ISO1541D, U3 ATTINY85-20SU, U4 ACPL-217-50DE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

Commit message: Added ibom for addon board, and put the elfa+RS components into the parts/ibom
Parts:
- C10, C3, C6, C7: elfa# (none) -> 300-87-136
- C11, C2, C5, C8, C9: elfa# (none) -> 301-11-165
- D1: elfa# (none) -> 170-02-190
- J1, J2: elfa# (none) -> 300-93-649
- J3: elfa# (none) -> 300-93-664
- J4: elfa# (none) -> 300-93-645
- R1, R3: elfa# (none) -> 300-37-977
- R10, R11, R7, R8, R9: value 4k7 -> 4K7
- R12: elfa# (none) -> 300-37-950
- R13: value 10k -> 10K; elfa# (none) -> 300-47-287
- R14: value 1k -> 1K; elfa# (none) -> 160-15-663
- R2: elfa# (none) -> 160-30-965
- R4: elfa# (none) -> 300-47-287
- R5, R6: value 470k -> 470K; elfa# (none) -> 300-37-953
- U1: RS# (none) -> 817-6580
- U2: RS# (none) -> 825-3075; elfa# (none) -> 300-22-572
- U3: elfa# (none) -> 173-21-927
- U6: RS# (none) -> 680-7131
- U8: RS# (none) -> 775-7450
