File: C64 Saver Throughhole 2.6/C64Saver2.kicad_pcb (KiCad board)
At the start: 2 copper layers, 43.9 x 28.8 mm, 24 parts, among them J1 Conn_01x04, J2 Conn_01x08, J4 Conn_01x08, J5 Conn_01x04, J6 Conn_01x04, Q1 BC547, Q2 IRFR5305

Commit message: Updated Throughole version (2.6). Gerbers, BOM, PDF etc. Moved old versions to folders. Might remove later
Parts:
- removed D1: TL431LP, TO_SOT_Packages_THT:TO-92_Inline_Narrow_Oval
- removed D3: 6V8, Diodes_THT:D_DO-35_SOD27_P7.62mm_Horizontal
- added U1: TL431LP, Package_TO_SOT_THT:TO-92_Inline, F.Cu at (165.1, 98.0)
- added Z1: 6V8, Diode_THT:D_DO-35_SOD27_P7.62mm_Horizontal, F.Cu at (153.4, 107.6)
- R1: value 3k9 -> 3k9 1%
- R2: value 3k3 -> 3k3 1%
- R3, R4, R5, R6: footprint Resistors_THT:R_Axial_DIN0204_L3.6mm_D1.6mm_P5.08mm_Horizontal -> Resistor_THT:R_Axial_DIN0204_L3.6mm_D1.6mm_P5.08mm_Horizontal
- moved J1 0.25 mm to (180.3, 108.2)
