File: C64 Saver Throughhole 2.6/C64Saver2.kicad_sch (KiCad schematic)
At the start: 24 parts, among them J1 Conn_01x04, J2 Conn_01x08, J4 Conn_01x08, J5 Conn_01x04, J6 Conn_01x04, Q1 BC547, Q2 IRFR5305

Commit message: SMD version 2.6 layout and schematics. Both THT and SMD are now on same version. should have same references.
Parts:
- renumbered D1 to U1, D3 to Z1
Other:
- note removed: "2018-09-23"
- note removed: "C64 Saver"
- title: (none) -> C64 Saver2 THT
Changed lines of the file:
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@@
 (kicad_sch (version 20230121) (generator eeschema)
   (paper "A4")
+  (title_block
+    (title "C64 Saver2 THT")
+    (date "2023-03-20")
+    (rev "2.6")
+  )
   (junction (at 91.44 137.16) (diameter 0) (color 0 0 0 0)
   )
@@
   (wire (pts (xy 91.44 124.46) (xy 91.44 137.16))
     (stroke (width 0) (type default))
-  )
-  (text "2018-09-23" (at 208.28 194.31 0)
-    (effects (font (size 2.0066 2.0066)) (justify left bottom))
   )
   (text "2.4" (at 269.24 194.31 0)
     (effects (font (size 1.524 1.524)) (justify left bottom))
   )
-  (text "C64 Saver" (at 187.96 190.5 0)
-    (effects (font (size 2.0066 2.0066)) (justify left bottom))
-  )
-  (label "VCC1+" (at 50.8 68.58 0)
-    (effects (font (size 1.2446 1.2446)) (justify left bottom))
-  )
-  (label "NGATE" (at 135.89 99.06 0)
-    (effects (font (size 1.2446 1.2446)) (justify left bottom))
-  )
-  (label "9VAC1" (at 77.47 124.46 0)
-    (effects (font (size 1.2446 1.2446)) (justify left bottom))
-  )
-  (label "SENSE" (at 90.805 104.14 0)
-    (effects (font (size 1.2446 1.2446)) (justify left bottom))
-  )
-  (label "9VAC1'" (at 96.52 124.46 0)
-    (effects (font (size 1.2446 1.2446)) (justify left bottom))
-  )
-  (label "9VAC2" (at 107.95 143.51 90)
-    (effects (font (size 1.2446 1.2446)) (justify left bottom))
-  )
-  (label "5V_SAFE" (at 153.67 68.58 0)
-    (effects (font (size 1.2446 1.2446)) (justify left bottom))
-  )
-  (label "VCC1-" (at 85.09 68.58 0)
-    (effects (font (size 1.2446 1.2446)) (justify left bottom))
-  )
-  (label "9VAC2" (at 78.74 121.92 0)
+  (label "VCC1+" (at 50.8 68.58 0) (fields_autoplaced)
+    (effects (font (size 1.2446 1.2446)) (justify left bottom))
+  )
+  (label "NGATE" (at 135.89 99.06 0) (fields_autoplaced)
+    (effects (font (size 1.2446 1.2446)) (justify left bottom))
+  )
+  (label "9VAC1" (at 77.47 124.46 0) (fields_autoplaced)
+    (effects (font (size 1.2446 1.2446)) (justify left bottom))
+  )
+  (label "SENSE" (at 90.805 104.14 0) (fields_autoplaced)
+    (effects (font (size 1.2446 1.2446)) (justify left bottom))
+  )
+  (label "9VAC1'" (at 96.52 124.46 0) (fields_autoplaced)
+    (effects (font (size 1.2446 1.2446)) (justify left bottom))
+  )
+  (label "9VAC2" (at 107.95 143.51 90) (fields_autoplaced)
+    (effects (font (size 1.2446 1.2446)) (justify left bottom))
+  )
+  (label "5V_SAFE" (at 153.67 68.58 0) (fields_autoplaced)
+    (effects (font (size 1.2446 1.2446)) (justify left bottom))
+  )
+  (label "VCC1-" (at 85.09 68.58 0) (fields_autoplaced)
+    (effects (font (size 1.2446 1.2446)) (justify left bottom))
+  )
+  (label "9VAC2" (at 78.74 121.92 0) (fields_autoplaced)
     (effects (font (size 1.2446 1.2446)) (justify left bottom))
   )
@@
   (symbol (lib_id "C64Saver2-rescue:D_Zener_Small") (at 139.7 73.66 270) (unit 1)
     (in_bom yes) (on_board yes) (dnp no)
-    (property "Reference" "D3" (at 141.986 73.66 0)
+    (property "Reference" "Z1" (at 141.986 73.66 0)
       (effects (font (size 1.27 1.27)))
     )
@@
       (project "C64Saver2"
         (path "/6fa111c1-4f39-4e94-92b0-76a2e6fa9f8e"
-          (reference "D3") (unit 1)
+          (reference "Z1") (unit 1)
         )
       )
@@
   (symbol (lib_id "C64Saver2-rescue:TL431LP") (at 99.695 104.14 90) (unit 1)
     (in_bom yes) (on_board yes) (dnp no)
-    (property "Reference" "D1" (at 97.155 106.68 0)
+    (property "Reference" "U1" (at 97.155 106.68 0)
       (effects (font (size 1.27 1.27)))
     )
@@
       (project "C64Saver2"
         (path "/6fa111c1-4f39-4e94-92b0-76a2e6fa9f8e"
-          (reference "D1") (unit 1)
-        )
-      )
+          (reference "U1") (unit 1)
+        )
+      )

Commit message: Updated Throughole version (2.6). Gerbers, BOM, PDF etc. Moved old versions to folders. Might remove later
Parts:
- removed U1: TL431LP, TO_SOT_Packages_THT:TO-92_Inline_Narrow_Oval, symbol C64Saver2-rescue:TL431LP
- added U1: TL431LP, Package_TO_SOT_THT:TO-92_Inline, symbol Reference_Voltage:TL431LP
- C1: kessler (none) -> 572309;0
- J1, J6: Mouser (none) -> not used
- LED1: Mouser (none) -> WP710A10LSECK/J3; kessler (none) -> 513513;0
- LED2: Mouser (none) -> WP710A10LZGCK; kessler (none) -> 513512;0
- MK1, MK2: Mouser (none) -> -; kessler (none) -> -; now left out of the parts list
- Q1: kessler (none) -> 500326;0
- Q2: kessler (none) -> 503060;0
- R1: value 3k9 -> 3k9 1%; kessler (none) -> 550563;0
- R10, R9: kessler (none) -> 550549;0
- R2: value 3k3 -> 3k3 1%; Mouser (none) -> RN55D3301FB14; kessler (none) -> 550561;0
- R3, R5: footprint Resistors_THT:R_Axial_DIN0204_L3.6mm_D1.6mm_P5.08mm_Horizontal -> Resistor_THT:R_Axial_DIN0204_L3.6mm_D1.6mm_P5.08mm_Horizontal; Mouser (none) -> RN55D3301FB14; kessler (none) -> 550561;0
- R4: footprint Resistors_THT:R_Axial_DIN0204_L3.6mm_D1.6mm_P5.08mm_Horizontal -> Resistor_THT:R_Axial_DIN0204_L3.6mm_D1.6mm_P5.08mm_Horizontal; kessler (none) -> 550609;0
- R6: footprint Resistors_THT:R_Axial_DIN0204_L3.6mm_D1.6mm_P5.08mm_Horizontal -> Resistor_THT:R_Axial_DIN0204_L3.6mm_D1.6mm_P5.08mm_Horizontal; kessler (none) -> 550563;0
- R7: footprint Resistors_THT:R_Axial_DIN0204_L3.6mm_D1.6mm_P5.08mm_Horizontal -> Resistor_THT:R_Axial_DIN0207_L6.3mm_D2.5mm_P7.62mm_Horizontal; kessler (none) -> 550585;0
- R8: footprint Resistor_THT:R_Axial_DIN0207_L6.3mm_D2.5mm_P7.62mm_Horizontal -> Resistor_THT:R_Axial_DIN0204_L3.6mm_D1.6mm_P5.08mm_Horizontal; kessler (none) -> 550573;0
- Z1: footprint Diodes_THT:D_DO-35_SOD27_P7.62mm_Horizontal -> Diode_THT:D_DO-35_SOD27_P7.62mm_Horizontal; kessler (none) -> 511511;0
Connections:
- net GND: now also U1.2 (A)
- net SENSE: now also U1.1 (REF)
- net at R3.2, R7.1, R9.2: now also U1.3 (K)
Other:
- moved on the sheet: J6, LED1, LED2, Q1, Q2, R10, R3, R4, R5, R6, R7, R8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

Commit message: Preparing for Saver 2.6, moving 2.5 and 2.4 to oldfiles folder
Other:
- moved on the sheet: J1, J2, J4, J5, J6, LED1, LED2, Q2, R1, R10, R3, R4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
